File: PWR_Supply/ 9V stabilizēts spriegums.sch (KiCad schematic (older format))
At the start: 3 parts, among them U2 LM7809_TO220

Commit message: Tresais majas darbs
Parts:
- C4, C5: Voltage (none) -> 50V
Changed lines of the file:
@@
 F 2 "" H 4900 3550 50  0001 C CNN
 F 3 "~" H 4900 3550 50  0001 C CNN
+F 4 "50V" H 4650 3550 50  0000 L CNN "Voltage"
 	1    4900 3550
 	1    0    0    -1
@@
 F 2 "" H 6400 3550 50  0001 C CNN
 F 3 "~" H 6400 3550 50  0001 C CNN
+F 4 "50V" H 6300 3550 50  0000 R CNN "Voltage"
 	1    6400 3550
 	1    0    0    -1
@@
 VCC
 Wire Wire Line
-	4900 3300 4500 3300
+	4900 3300 4700 3300
 Connection ~ 4900 3300
 Text HLabel 7050 3300 2    50   Input ~ 0
@@
 Wire Wire Line
 	5700 3700 5700 3850
+$Comp
+L power:PWR_FLAG #FLG0102
+U 1 1 5F860B9C
+P 4700 3300
+F 0 "#FLG0102" H 4700 3375 50  0001 C CNN
+F 1 "PWR_FLAG" H 4700 3473 50  0000 C CNN
+F 2 "" H 4700 3300 50  0001 C CNN
+F 3 "~" H 4700 3300 50  0001 C CNN
+	1    4700 3300
+	1    0    0    -1
+$EndComp
+Connection ~ 4700 3300
+Wire Wire Line
+	4700 3300 4500 3300
 $EndSCHEMATC
