File: PWR_Supply/12V stabilizēts spriegums.sch (KiCad schematic (older format))
At the start: 3 parts, among them U3 LM7812_TO220

Commit message: Tresais majas darbs
Parts:
- C6, C7: Voltage (none) -> 50V
Changed lines of the file:
@@
 $Descr A4 11693 8268
 encoding utf-8
-Sheet 6 6
+Sheet 5 6
 Title ""
 Date ""
@@
 F 2 "" H 5000 3500 50  0001 C CNN
 F 3 "~" H 5000 3500 50  0001 C CNN
+F 4 "50V" H 4900 3500 50  0000 R CNN "Voltage"
 	1    5000 3500
 	1    0    0    -1
@@
 F 2 "" H 6250 3500 50  0001 C CNN
 F 3 "~" H 6250 3500 50  0001 C CNN
+F 4 "50V" H 6150 3500 50  0000 R CNN "Voltage"
 	1    6250 3500
 	1    0    0    -1
