File: PWR_Supply/3,3V stabilizēts spriegums.sch (KiCad schematic (older format))
At the start: 3 parts, among them U4 LM1084-3.3

Commit message: Tresais majas darbs
Parts:
- C8, C9: Voltage (none) -> 50V
Changed lines of the file:
@@
 F 2 "" H 4550 3150 50  0001 C CNN
 F 3 "~" H 4550 3150 50  0001 C CNN
+F 4 "50V" H 4450 3150 50  0000 R CNN "Voltage"
 	1    4550 3150
 	1    0    0    -1
@@
 F 2 "" H 6150 3150 50  0001 C CNN
 F 3 "~" H 6150 3150 50  0001 C CNN
+F 4 "50V" H 6050 3150 50  0000 R CNN "Voltage"
 	1    6150 3150
 	1    0    0    -1
