File: PWR_Supply/5V stabilizēts spriegums.sch (KiCad schematic (older format))
At the start: 3 parts, among them U1 L7805

Commit message: Tresais majas darbs
Parts:
- C2, C3: Voltage (none) -> 50V
Changed lines of the file:
@@
 F 2 "" H 4600 3500 50  0001 C CNN
 F 3 "~" H 4600 3500 50  0001 C CNN
+F 4 "50V" H 4350 3500 50  0000 L CNN "Voltage"
 	1    4600 3500
 	1    0    0    -1
@@
 F 2 "" H 6500 3500 50  0001 C CNN
 F 3 "~" H 6500 3500 50  0001 C CNN
+F 4 "50V" H 6400 3500 50  0000 R CNN "Voltage"
 	1    6500 3500
 	1    0    0    -1
@@
 $EndComp
 Wire Wire Line
-	5500 3700 5500 3900
+	5500 3700 5500 3850
 Text HLabel 4150 3250 0    50   Input ~ 0
 VCC
@@
 	4600 3700 4150 3700
 Connection ~ 4600 3700
+$Comp
+L power:PWR_FLAG #FLG0101
+U 1 1 5F86008A
+P 5500 3850
+F 0 "#FLG0101" H 5500 3925 50  0001 C CNN
+F 1 "PWR_FLAG" V 5500 3978 50  0000 L CNN
+F 2 "" H 5500 3850 50  0001 C CNN
+F 3 "~" H 5500 3850 50  0001 C CNN
+	1    5500 3850
+	0    1    1    0
+$EndComp
+Connection ~ 5500 3850
+Wire Wire Line
+	5500 3850 5500 3900
 $EndSCHEMATC
