File: Battery/Battery.sch (KiCad schematic (older format))
At the start: 2 parts

Commit message: Piektais majas darbs
Parts:
- added BT3: 1072TR, Battery_Holder:1072TR, symbol Device:Battery_Cell
- added BT4: 1060, Battery_Holder:1060, symbol Device:Battery_Cell
- added BT5: 2992, Battery_Holder:2992, symbol Device:Battery_Cell
Connections:
- net +5V: now also BT3.1 (+), BT4.1 (+), BT5.1 (+)
- net GND: now also BT3.2 (-), BT4.2 (-), BT5.2 (-)
Changed lines of the file:
@@
 Wire Wire Line
 	6400 2950 6400 2650
+$Comp
+L Device:Battery_Cell BT3
+U 1 1 5F984D7F
+P 7150 3150
+F 0 "BT3" H 7268 3246 50  0000 L CNN
+F 1 "1072TR" H 7268 3155 50  0000 L CNN
+F 2 "Battery_Holder:1072TR" V 7150 3210 50  0001 C CNN
+F 3 "~" V 7150 3210 50  0001 C CNN
+	1    7150 3150
+	1    0    0    -1
+$EndComp
+$Comp
+L Device:Battery_Cell BT4
+U 1 1 5F986107
+P 7850 3150
+F 0 "BT4" H 7968 3246 50  0000 L CNN
+F 1 "1060" H 7968 3155 50  0000 L CNN
+F 2 "Battery_Holder:1060" V 7850 3210 50  0001 C CNN
+F 3 "~" V 7850 3210 50  0001 C CNN
+	1    7850 3150
+	1    0    0    -1
+$EndComp
+$Comp
+L Device:Battery_Cell BT5
+U 1 1 5F98688A
+P 8550 3150
+F 0 "BT5" H 8668 3246 50  0000 L CNN
+F 1 "2992" H 8668 3155 50  0000 L CNN
+F 2 "Battery_Holder:2992" V 8550 3210 50  0001 C CNN
+F 3 "~" V 8550 3210 50  0001 C CNN
+	1    8550 3150
+	1    0    0    -1
+$EndComp
+Wire Wire Line
+	6400 3250 7150 3250
+Connection ~ 6400 3250
+Connection ~ 7150 3250
+Wire Wire Line
+	7150 3250 7850 3250
+Connection ~ 7850 3250
+Wire Wire Line
+	7850 3250 8550 3250
+$Comp
+L power:+5V #PWR04
+U 1 1 5F9873BC
+P 7150 2650
+F 0 "#PWR04" H 7150 2500 50  0001 C CNN
+F 1 "+5V" H 7165 2823 50  0000 C CNN
+F 2 "" H 7150 2650 50  0001 C CNN
+F 3 "" H 7150 2650 50  0001 C CNN
+	1    7150 2650
+	1    0    0    -1
+$EndComp
+$Comp
+L power:+5V #PWR05
+U 1 1 5F9877A7
+P 7850 2700
+F 0 "#PWR05" H 7850 2550 50  0001 C CNN
+F 1 "+5V" H 7865 2873 50  0000 C CNN
+F 2 "" H 7850 2700 50  0001 C CNN
+F 3 "" H 7850 2700 50  0001 C CNN
+	1    7850 2700
+	1    0    0    -1
+$EndComp
+$Comp
+L power:+5V #PWR06
+U 1 1 5F987B48
+P 8550 2700
+F 0 "#PWR06" H 8550 2550 50  0001 C CNN
+F 1 "+5V" H 8565 2873 50  0000 C CNN
+F 2 "" H 8550 2700 50  0001 C CNN
+F 3 "" H 8550 2700 50  0001 C CNN
+	1    8550 2700
+	1    0    0    -1
+$EndComp
+Wire Wire Line
+	7150 2650 7150 2950
+Wire Wire Line
+	7850 2700 7850 2950
+Wire Wire Line
+	8550 2700 8550 2950
 $EndSCHEMATC

Commit message: Sestais majas darbs
Parts:
- BT2: footprint (none) -> Battery_Holder:S8211R
Changed lines of the file:
@@
 F 0 "BT2" H 6518 3246 50  0000 L CNN
 F 1 "S8211R" H 6518 3155 50  0000 L CNN
-F 2 "" V 6400 3210 50  0001 C CNN
+F 2 "Battery_Holder:S8211R" V 6400 3210 50  0001 C CNN
 F 3 "~" V 6400 3210 50  0001 C CNN
 	1    6400 3150
