File: Single_transistor_AMP/Single_transistor_AMP.kicad_pcb (KiCad board)
At the start: 2 copper layers, 0 parts

Commit message: Septitajs majas darbs
Parts:
- added C1: 1uF, Capacitor_SMD:C_0805_2012Metric, F.Cu at (120.9, 79.2)
- added C2: 10uF, Capacitor_SMD:CP_Elec_4x3, F.Cu at (131.8, 84.8)
- added C3: 1uF, Capacitor_SMD:C_0805_2012Metric, F.Cu at (156.3, 84.8)
- added J1: Signal_Input, Connector_PinHeader_2.54mm:PinHeader_1x02_P2.54mm_Vertical, F.Cu at (116.8, 86.4)
- added J2: +12V, Connector_PinHeader_2.54mm:PinHeader_1x02_P2.54mm_Vertical, F.Cu at (146.3, 89.4)
- added J3: Signal_Output, Connector_PinHeader_2.54mm:PinHeader_1x02_P2.54mm_Vertical, F.Cu at (155.2, 89.4)
- added Q1: 2N3904, Package_TO_SOT_THT:TO-92_Inline, F.Cu at (125.5, 79.2)
- added Q2: 2N3904, Package_TO_SOT_THT:TO-92_Inline, F.Cu at (144.3, 79.0)
- added R1: 10k, Resistor_SMD:R_0805_2012Metric_Pad1.20x1.40mm_HandSolder, F.Cu at (125.6, 84.8)
- added R2: 220k, Resistor_SMD:R_0805_2012Metric_Pad1.20x1.40mm_HandSolder, F.Cu at (147.2, 84.8)
- added R3: 1k, Resistor_SMD:R_0805_2012Metric_Pad1.20x1.40mm_HandSolder, F.Cu at (121.0, 85.0)
- added R4: 100k, Resistor_SMD:R_0805_2012Metric_Pad1.20x1.40mm_HandSolder, F.Cu at (137.9, 84.8)
- added R5: 6.8k, Resistor_SMD:R_0805_2012Metric_Pad1.20x1.40mm_HandSolder, F.Cu at (151.9, 84.8)
- added R6: 1k, Resistor_SMD:R_0805_2012Metric_Pad1.20x1.40mm_HandSolder, F.Cu at (142.5, 84.8)
Other:
- board outline added: 53.4 x 21.9 mm

Commit message: Astotais majas darbs
Routing:
- net Net-(Q1-Pad3): track 0.00 -> 24.6 mm
- net Net-(C2-Pad1): track 0.00 -> 14.6 mm
- net Net-(C3-Pad2): track 0.00 -> 11.6 mm
- net Net-(C1-Pad1): track 0.00 -> 11.4 mm
- net Net-(Q2-Pad1): track 0.00 -> 10.2 mm
- net Net-(J2-Pad1): track 0.00 -> 8.64 mm
- net Net-(Q1-Pad1): track 0.00 -> 6.56 mm
- net Net-(C1-Pad2): track 0.00 -> 5.86 mm
- net Net-(C3-Pad1): track 0.00 -> 4.10 mm
- added copper zone on F.Cu, net (none)
- added copper zone on B.Cu, net GND
- added copper zone on F.Cu, net GND
Changed lines of the file:
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@@
     (thickness 1.6)
     (drawings 5)
-    (tracks 0)
+    (tracks 32)
     (zones 0)
     (modules 14)
@@
   (setup
     (last_trace_width 0.25)
+    (user_trace_width 0.5)
+    (user_trace_width 0.75)
     (trace_clearance 0.2)
     (zone_clearance 0.508)
@@
     (uvia_dia 0.3)
     (uvia_drill 0.1)
-    (add_net GND)
     (add_net "Net-(C1-Pad1)")
     (add_net "Net-(C1-Pad2)")
     (add_net "Net-(C2-Pad1)")
-    (add_net "Net-(C3-Pad1)")
     (add_net "Net-(C3-Pad2)")
     (add_net "Net-(J2-Pad1)")
@@
     (uvia_dia 0.3)
     (uvia_drill 0.1)
+    (add_net GND)
+    (add_net "Net-(C3-Pad1)")
   )
   (module Capacitor_SMD:C_0805_2012Metric (layer F.Cu)
@@
       (effects (font (size 1 1) (thickness 0.15)))
     )
-    (fp_text user %R (at 0 1.27 90) (layer F.Fab)
-      (effects (font (size 1 1) (thickness 0.15)))
-    )
     (fp_line (start -0.635 -1.27) (end 1.27 -1.27) (layer F.Fab) (width 0.1))
     (fp_line (start 1.27 -1.27) (end 1.27 3.81) (layer F.Fab) (width 0.1))
@@
     (fp_line (start 1.8 4.35) (end 1.8 -1.8) (layer F.CrtYd) (width 0.05))
     (fp_line (start 1.8 -1.8) (end -1.8 -1.8) (layer F.CrtYd) (width 0.05))
+    (fp_text user %R (at 0 1.27 90) (layer F.Fab)
+      (effects (font (size 1 1) (thickness 0.15)))
+    )
     (pad 2 thru_hole oval (at 0 2.54 180) (size 1.7 1.7) (drill 1) (layers *.Cu *.Mask)
       (net 2 "Net-(C1-Pad2)"))
@@
   (gr_line (start 109.675588 79.15777) (end 109.6772 91.6813) (layer Edge.Cuts) (width 0.05))
   (gr_arc (start 136.144 135.255) (end 163.067999 79.375001) (angle -50.98500316) (layer Edge.Cuts) (width 0.05))
+  (segment (start 126.746 82.693) (end 126.746 79.248) (width 0.5) (layer F.Cu) (net 1))
+  (segment (start 125.603 83.836) (end 126.746 82.693) (width 0.5) (layer F.Cu) (net 1))
+  (segment (start 126.746 78.432998) (end 126.746 79.248) (width 0.5) (layer F.Cu) (net 1))
+  (segment (start 126.361001 78.047999) (end 126.746 78.432998) (width 0.5) (layer F.Cu) (net 1))
+  (segment (start 123.054001 78.047999) (end 126.361001 78.047999) (width 0.5) (layer F.Cu) (net 1))
+  (segment (start 121.854 79.248) (end 123.054001 78.047999) (width 0.5) (layer F.Cu) (net 1))
+  (segment (start 116.84 82.362) (end 119.954 79.248) (width 0.5) (layer F.Cu) (net 2))
+  (segment (start 116.84 83.82) (end 116.84 82.362) (width 0.5) (layer F.Cu) (net 2))
+  (segment (start 129.026 85.836) (end 131.826 83.036) (width 0.5) (layer F.Cu) (net 3))
+  (segment (start 125.603 85.836) (end 129.026 85.836) (width 0.5) (layer F.Cu) (net 3))
+  (segment (start 135.122 83.036) (end 137.922 85.836) (width 0.5) (layer F.Cu) (net 3))
+  (segment (start 131.826 83.036) (end 135.122 83.036) (width 0.5) (layer F.Cu) (net 3))
+  (segment (start 156.287 83.836) (end 156.337 83.886) (width 0.5) (layer F.Cu) (net 5))
+  (segment (start 151.892 83.836) (end 156.287 83.836) (width 0.5) (layer F.Cu) (net 5))
+  (segment (start 147.05 78.994) (end 151.892 83.836) (width 0.5) (layer F.Cu) (net 5))
+  (segment (start 146.812 78.994) (end 147.05 78.994) (width 0.5) (layer F.Cu) (net 5))
+  (segment (start 155.194 86.929) (end 156.337 85.786) (width 0.5) (layer F.Cu) (net 6))
+  (segment (start 155.194 89.408) (end 155.194 86.929) (width 0.5) (layer F.Cu) (net 6))
+  (segment (start 146.304 86.725) (end 147.193 85.836) (width 0.5) (layer F.Cu) (net 7))
+  (segment (start 146.304 89.408) (end 146.304 86.725) (width 0.5) (layer F.Cu) (net 7))
+  (segment (start 147.193 85.836) (end 151.892 85.836) (width 0.5) (layer F.Cu) (net 7))
+  (segment (start 145.542 82.185) (end 147.193 83.836) (width 0.5) (layer F.Cu) (net 8))
+  (segment (start 145.542 78.994) (end 145.542 82.185) (width 0.5) (layer F.Cu) (net 8))
+  (segment (start 145.542 78.178998) (end 145.542 78.994) (width 0.5) (layer F.Cu) (net 8))
+  (segment (start 145.157001 77.793999) (end 145.542 78.178998) (width 0.5) (layer F.Cu) (net 8))
+  (segment (start 129.470001 77.793999) (end 145.157001 77.793999) (width 0.5) (layer F.Cu) (net 8))
+  (segment (start 128.016 79.248) (end 129.470001 77.793999) (width 0.5) (layer F.Cu) (net 8))
+  (segment (start 121.031 83.693) (end 125.476 79.248) (width 0.5) (layer F.Cu) (net 9))
+  (segment (start 121.031 83.963) (end 121.031 83.693) (width 0.5) (layer F.Cu) (net 9))
+  (segment (start 137.922 83.836) (end 142.494 83.836) (width 0.5) (layer F.Cu) (net 10))
+  (segment (start 142.494 80.772) (end 144.272 78.994) (width 0.5) (layer F.Cu) (net 10))
+  (segment (start 142.494 83.836) (end 142.494 80.772) (width 0.5) (layer F.Cu) (net 10))
+  (zone (net 4) (net_name GND) (layer F.Cu) (hatch edge 0.508)
+    (connect_pads (clearance 0.508))
+    (min_thickness 0.254)
+    (fill yes (arc_segments 32) (thermal_gap 0.508) (thermal_bridge_width 0.508))
+    (polygon
+      (pts
+        (xy 138.85 73.3) (xy 142.2 73.525) (xy 145.85 74) (xy 148.925 74.55) (xy 152.25 75.375)
+        (xy 154.675 76.075) (xy 156.525 76.675) (xy 158.025 77.225) (xy 159.325 77.725) (xy 160.375 78.15)
+        (xy 161.55 78.675) (xy 163.075 79.375) (xy 163.075 95.15) (xy 109.675 95.15) (xy 109.675 79.175)
+        (xy 111.575 78.3) (xy 115.45 76.8) (xy 119.6 75.475) (xy 123.025 74.625) (xy 128.2 73.75)
+        (xy 131.175 73.425) (xy 134.975 73.25)
+      )
+    )
+  )
+  (zone (net 0) (net_name "") (layer F.Cu) (hatch edge 0.508)
+    (priority 2)
+    (connect_pads (clearance 0.508))
+    (min_thickness 0.254)
+    (fill yes (arc_segments 32) (thermal_gap 0.508) (thermal_bridge_width 0.508))
+    (polygon
+      (pts
+        (xy 133.45 81.15) (xy 130.525 81.15) (xy 130.375 82.35) (xy 129.075 85.25) (xy 126.625 85.425)
+        (xy 127.125 83.65) (xy 127.225 80.65) (xy 128.55 80.25) (xy 129.775 78.575) (xy 133.475 78.325)
+      )
+    )
+  )
+  (zone (net 0) (net_name "") (layer F.Cu) (hatch edge 0.508)
+    (priority 3)
+    (connect_pads (clearance 0.508))
+    (min_thickness 0.254)
+    (fill yes (arc_segments 32) (thermal_gap 0.508) (thermal_bridge_width 0.508))
+    (polygon
+      (pts
+        (xy 143.225 79.3) (xy 142.025 80.675) (xy 142 83) (xy 136.25 83.2) (xy 134.75 82.375)
+        (xy 133.125 82.3) (xy 133.4 78.6) (xy 143.175 78.475)
+      )
+    )
+  )
+  (zone (net 0) (net_name "") (layer F.Cu) (hatch edge 0.508)
+    (priority 3)
+    (connect_pads (clearance 0.508))
+    (min_thickness 0.254)
+    (fill yes (arc_segments 32) (thermal_gap 0.508) (thermal_bridge_width 0.508))
+    (polygon
+      (pts
+        (xy 149.225 81.875) (xy 148.575 82.825) (xy 147.3 82.8) (xy 146.125 81.9) (xy 146.175 80.1)
+        (xy 147.125 80.025)
+      )
+    )
+  )
+  (zone (net 0) (net_name "") (layer F.Cu) (hatch edge 0.508)
+    (priority 4)
+    (connect_pads (clearance 0.508))
+    (min_thickness 0.254)
+    (fill yes (arc_segments 32) (thermal_gap 0.508) (thermal_bridge_width 0.508))
+    (polygon
+      (pts
+        (xy 150.825 83.425) (xy 150.775 85.425) (xy 148.25 85.45) (xy 148.275 82.8) (xy 149.2 81.85)
+      )
+    )
+  )
+  (zone (net 4) (net_name GND) (layer B.Cu) (hatch edge 0.508)
+    (connect_pads (clearance 0.508))
+    (min_thickness 0.254)
+    (fill yes (arc_segments 32) (thermal_gap 0.508) (thermal_bridge_width 0.508))
+    (polygon
+      (pts
+        (xy 152.25 75.35) (xy 163.075 79.375) (xy 163.075 95.15) (xy 109.675 95.15) (xy 109.675 79.175)
+        (xy 114.2 77.225) (xy 125.475 74.25) (xy 139.55 73.325)
+      )
+    )
+  )
 )
