File: Single_transistor_AMP/Single_transistor_AMP.sch (KiCad schematic (older format))
At the start: 14 parts, among them J1 Signal_Input, J2 +12V, J3 Signal_Output, Q1 2N3904, Q2 2N3904

Commit message: Astotais majas darbs
Parts:
- J1, J2, J3: footprint Connector_AMASS:AMASS_XT30U-F_1x02_P5.0mm_Vertical -> Connector_PinHeader_2.54mm:PinHeader_1x02_P2.54mm_Vertical
Changed lines of the file:
@@
 F 0 "J3" H 5800 2950 50  0000 L CNN
 F 1 "Signal_Output" V 5950 2550 50  0000 L CNN
-F 2 "Connector_AMASS:AMASS_XT30U-F_1x02_P5.0mm_Vertical" H 5850 2850 50  0001 C CNN
+F 2 "Connector_PinHeader_2.54mm:PinHeader_1x02_P2.54mm_Vertical" H 5850 2850 50  0001 C CNN
 F 3 "~" H 5850 2850 50  0001 C CNN
 	1    5850 2850
@@
 F 0 "J1" H 3200 3350 50  0000 C CNN
 F 1 "Signal_Input" V 3300 3500 50  0000 C CNN
-F 2 "Connector_AMASS:AMASS_XT30U-F_1x02_P5.0mm_Vertical" H 3200 3550 50  0001 C CNN
+F 2 "Connector_PinHeader_2.54mm:PinHeader_1x02_P2.54mm_Vertical" H 3200 3550 50  0001 C CNN
 F 3 "~" H 3200 3550 50  0001 C CNN
 	1    3200 3550
@@
 F 0 "J2" H 5250 2150 50  0000 L CNN
 F 1 "+12V" V 5400 1900 50  0000 L CNN
-F 2 "Connector_AMASS:AMASS_XT30U-F_1x02_P5.0mm_Vertical" H 5300 2050 50  0001 C CNN
+F 2 "Connector_PinHeader_2.54mm:PinHeader_1x02_P2.54mm_Vertical" H 5300 2050 50  0001 C CNN
 F 3 "~" H 5300 2050 50  0001 C CNN
 	1    5300 2050
